File: hardware/zero3-carrier/zero3-water-logger-carrier.kicad_pcb (KiCad board)
At the start: 2 copper layers, 160 x 100 mm, 19 parts, among them J1 Orange Pi Zero 3 26-pin header, J10 Turbidity sensor, J11 ORP sensor, J12 DO sensor, J13 NH4 ISE amp, J14 5V load switch reserved, J2 Raspberry Pi Pico socket, J3 ADS1115 #1 0x48, J4 ADS1115 #2 0x49, J5 DS18B20, J6 BME280, J7 DS3231 RTC, J8 pH sensor, J9 TDS sensor

Commit message: Add schematic synced Zero 3 carrier PCB draft
Parts:
- added C1: 470uF-1000uF 10V, CP_Radial_D10.0mm_P5.00mm, F.Cu at (315.0, 47.0)
- added CBOOT: 100nF, C_0603_1608Metric, F.Cu at (200.0, 82.0)
- added CCOMP1: 2200pF, C_0603_1608Metric, F.Cu at (245.0, 97.0)
- added CCOMP2: 22pF, C_0603_1608Metric, F.Cu at (260.0, 97.0)
- added CIN1: 4.7uF 50V, C_1206_3216Metric, F.Cu at (160.0, 82.0)
- added CIN2: 4.7uF 50V, C_1206_3216Metric, F.Cu at (175.0, 82.0)
- added CIN3: 10nF 50V, C_0603_1608Metric, F.Cu at (275.0, 97.0)
- added COUT1: 47uF 10V, C_1210_3225Metric, F.Cu at (245.0, 47.0)
- added COUT2: 47uF 10V, C_1210_3225Metric, F.Cu at (260.0, 47.0)
- added CSS: 10nF, C_0603_1608Metric, F.Cu at (215.0, 82.0)
- added D1: VBUS TVS, D_SMA, F.Cu at (73.0, 47.0)
- added D2: 5A 40V Schottky, D_SMA, F.Cu at (220.0, 62.0)
- added F1: 3A-5A polyfuse, Fuse_1206_3216Metric, F.Cu at (140.0, 47.0)
- added J15: Download button, PinHeader_1x04_P2.54mm_Vertical, F.Cu at (330.0, 127.0)
- added J16: Spare analog header, PinHeader_1x04_P2.54mm_Vertical, F.Cu at (330.0, 167.0)
- added L1: 4.7uH >=6A, L_10.4x10.4_H4.8, F.Cu at (220.0, 47.0)
- added Q1: AO4407A P-MOS high-side, SOIC-8_3.9x4.9mm_P1.27mm, F.Cu at (285.0, 47.0)
- added Q2: 2N7002, SOT-23, F.Cu at (285.0, 72.0)
- added R2: 100k, R_0603_1608Metric, F.Cu at (305.0, 57.0)
- added R3: 1k, R_0603_1608Metric, F.Cu at (305.0, 72.0)
- added R4: 100k, R_0603_1608Metric, F.Cu at (305.0, 84.0)
- added R5: 330R if 3.3V LED, R_0603_1608Metric, F.Cu at (330.0, 145.0)
- added RCOMP1: 37.4k, R_0603_1608Metric, F.Cu at (230.0, 97.0)
- added REN1: 665k, R_0603_1608Metric, F.Cu at (200.0, 97.0)
- added REN2: 130k, R_0603_1608Metric, F.Cu at (215.0, 97.0)
- added RFB1: 10.2k 1%, R_0603_1608Metric, F.Cu at (245.0, 70.0)
- added RFB2: 1.96k 1%, R_0603_1608Metric, F.Cu at (260.0, 70.0)
- added U1: CH224K PD sink 9V, SSOP-10_3.9x4.9mm_P1.00mm, F.Cu at (103.0, 47.0)
- added U2: TPS54531DDA 5A buck, TI_SO-PowerPAD-8, F.Cu at (180.0, 52.0)
- H1, H2, H3, H4: value MountingHole -> MountingHole_3.2mm_M3; footprint MountingHole_3.2mm -> MountingHole_3.2mm_M3
- J1: value Orange Pi Zero 3 26-pin header -> Orange Pi Zero 3 26-pin; footprint Zero3_2x13_Header -> PinHeader_2x13_P2.54mm_Vertical
- J10, J11, J13, J8, J9: footprint ScrewTerminal_1x03 -> TerminalBlock_Phoenix_MKDS-1,5-3-5.08_1x03_P5.08mm_Horizontal
- J12: value DO sensor -> Dissolved oxygen; footprint ScrewTerminal_1x03 -> TerminalBlock_Phoenix_MKDS-1,5-3-5.08_1x03_P5.08mm_Horizontal
- J14: value 5V load switch reserved -> USB-C PD input; footprint LoadSwitch_Reserved_1x05 -> USB_C_Receptacle_HRO_TYPE-C-31-M-12
- J2: footprint Pico_2x20_Socket -> RaspberryPi_Pico_Common_THT
- J3, J4: footprint ADS1115_Module_Header -> PinHeader_1x09_P2.54mm_Vertical
- J5: value DS18B20 -> DS18B20 water temp; footprint Module_1x03 -> PinHeader_1x03_P2.54mm_Vertical
- J6: value BME280 -> BME280 air sensor; footprint Module_1x04 -> PinHeader_1x04_P2.54mm_Vertical
- J7: footprint Module_1x04 -> PinHeader_1x04_P2.54mm_Vertical
- R1: value 4.7k DS18B20 pull-up -> 4.7k; footprint Resistor_THT_7.62mm -> R_Axial_DIN0207_L6.3mm_D2.5mm_P7.62mm_Horizontal
- moved H3 403.6 mm to (344.0, 314.0)
- moved H4 259.4 mm to (16.0, 314.0)
- moved J7 225.8 mm to (295.0, 127.0), turned to 90 degrees
- moved J8 205.3 mm to (45.0, 202.0), turned to 90 degrees
- moved J6 200.8 mm to (260.0, 127.0), turned to 90 degrees
- moved H2 189.3 mm to (344.0, 16.0)
- moved J9 179.4 mm to (85.0, 202.0), turned to 90 degrees
- moved J5 178.6 mm to (225.0, 127.0), turned to 90 degrees
- moved J13 165.1 mm to (245.0, 202.0), turned to 90 degrees
- moved R1 161.5 mm to (225.0, 145.0)
- moved J10 160.4 mm to (125.0, 202.0), turned to 90 degrees
- moved J12 152.5 mm to (205.0, 202.0), turned to 90 degrees
- moved J11 150.8 mm to (165.0, 202.0), turned to 90 degrees
- moved J4 133.3 mm to (185.0, 132.0), turned to 90 degrees
- moved J2 125.2 mm to (97.0, 137.0), turned to 90 degrees
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Connections:
- J1 pad 1: (no net) -> OPI_3V3
- J1 pad 10: (no net) -> UART_PICO_TX_OPI_RX
- J1 pad 11: (no net) -> OPI_READY
- J1 pad 14: (no net) -> GND
- J1 pad 17: (no net) -> OPI_3V3
- J1 pad 2: (no net) -> OPI_5V_SW
- J1 pad 20: (no net) -> GND
- J1 pad 25: (no net) -> GND
- J1 pad 3: (no net) -> OPI_SDA
- J1 pad 4: (no net) -> OPI_5V_SW
- J1 pad 5: (no net) -> OPI_SCL
- J1 pad 6: (no net) -> GND
- J1 pad 7: (no net) -> OPI_1WIRE
- J1 pad 8: (no net) -> UART_OPI_TX_PICO_RX
- J1 pad 9: (no net) -> GND
- J10 pad 1: (no net) -> OPI_5V_SW
- J10 pad 2: (no net) -> GND
- J10 pad 3: (no net) -> TURB_AIN
- J11 pad 1: (no net) -> OPI_5V_SW
- J11 pad 2: (no net) -> GND
- J11 pad 3: (no net) -> ORP_AIN
- J12 pad 1: (no net) -> OPI_5V_SW
- J12 pad 2: (no net) -> GND
- J12 pad 3: (no net) -> DO_AIN
- J13 pad 1: (no net) -> OPI_5V_SW
- J13 pad 2: (no net) -> GND
- J13 pad 3: (no net) -> NH4_AIN
- J2 pad 1: (no net) -> UART_PICO_TX_OPI_RX
- J2 pad 13: (no net) -> GND
- J2 pad 17: (no net) -> OPI_READY
- J2 pad 18: (no net) -> GND
- J2 pad 19: (no net) -> PICO_GP14
- J2 pad 2: (no net) -> UART_OPI_TX_PICO_RX
- J2 pad 20: (no net) -> PICO_GP15
- J2 pad 21: (no net) -> PICO_LED_GP16
- J2 pad 23: (no net) -> GND
- J2 pad 28: (no net) -> GND
- J2 pad 3: (no net) -> GND
- J2 pad 33: (no net) -> GND
- J2 pad 36: (no net) -> PICO_3V3
- J2 pad 38: (no net) -> GND
- J2 pad 39: (no net) -> FUSED_5V1
- J2 pad 6: (no net) -> PICO_GP4
- J2 pad 7: (no net) -> PICO_GP5
- J2 pad 8: (no net) -> GND
- J3 pad 1: (no net) -> OPI_3V3
- J3 pad 2: (no net) -> GND
- J3 pad 3: (no net) -> OPI_SDA
- J3 pad 4: (no net) -> OPI_SCL
- J3 pad 5: (no net) -> GND
- J3 pad 6: (no net) -> PH_AIN
- J3 pad 7: (no net) -> TDS_AIN
- J3 pad 8: (no net) -> TURB_AIN
- J3 pad 9: (no net) -> ORP_AIN
- J4 pad 1: (no net) -> OPI_3V3
- J4 pad 2: (no net) -> GND
- J4 pad 3: (no net) -> OPI_SDA
- J4 pad 4: (no net) -> OPI_SCL
- J4 pad 5: (no net) -> OPI_3V3
- J4 pad 6: (no net) -> DO_AIN
- J4 pad 7: (no net) -> NH4_AIN
- J4 pad 8: (no net) -> SPARE_AIN2
- J4 pad 9: (no net) -> SPARE_AIN3
- J5 pad 1: (no net) -> OPI_3V3
- J5 pad 2: (no net) -> OPI_1WIRE
- J5 pad 3: (no net) -> GND
- J6 pad 1: (no net) -> OPI_3V3
- J6 pad 2: (no net) -> GND
- J6 pad 3: (no net) -> OPI_SDA
- J6 pad 4: (no net) -> OPI_SCL
- J7 pad 1: (no net) -> PICO_3V3
- J7 pad 2: (no net) -> GND
- J7 pad 3: (no net) -> PICO_GP4
- J7 pad 4: (no net) -> PICO_GP5
- J8 pad 1: (no net) -> OPI_5V_SW
- J8 pad 2: (no net) -> GND
- J8 pad 3: (no net) -> PH_AIN
- J9 pad 1: (no net) -> OPI_5V_SW
- J9 pad 2: (no net) -> GND
- J9 pad 3: (no net) -> TDS_AIN
- R1 pad 1: (no net) -> OPI_3V3
- R1 pad 2: (no net) -> OPI_1WIRE
Other:
- board size 160 x 100 mm -> 344 x 314 mm
- board text removed: "ADS1115 modules and sensor terminals"
- board text removed: "Orange Pi Zero 3 header area"
- board text removed: "Pico socket"
- board text removed: "R0 PLACEMENT SKELETON - NOT READY TO ORDER"
