File: hardware/zero3-carrier/zero3-water-logger-carrier.kicad_pcb (KiCad board)
At the start: 2 copper layers, 344 x 314 mm, 48 parts, among them J1 Orange Pi Zero 3 26-pin, J10 Turbidity sensor, J11 ORP sensor, J12 Dissolved oxygen, J13 NH4 ISE amp, J14 USB-C PD input, J15 Download button, J16 Spare analog header, J2 Raspberry Pi Pico socket, J3 ADS1115 #1 0x48, J4 ADS1115 #2 0x49, J5 DS18B20 water temp, J6 BME280 air sensor, J7 DS3231 RTC, J8 pH sensor, J9 TDS sensor, Q1 AO4407A P-MOS high-side, Q2 2N7002, U1 CH224K PD sink 9V, U2 TPS54531DDA 5A buck

Commit message: Add GND pours, Freerouting wrapper, validator, manual routing guide
PCB:
- generate_pcb.py now adds filled GND copper pours on both layers with
  solid (non-thermal) pad connection. This brings unconnected-pad count
  down from 136 to 83 with zero DRC violations.

Tooling:
- route_with_freerouting.py: one-command auto-routing. Exports the PCB
  to Specctra DSN, fetches a pinned Freerouting JAR (v2.2.4) into
  ~/.cache/freerouting/, runs it headlessly, imports the SES, refills
  the GND pour, and re-runs DRC. Requires user authorization for
  external code execution on first run.
- validate_design.py: ERC + DRC + pinout-CSV format gate behind a
  single command. Currently passes (0 violations, 83 unconnected
  items noted but not a hard fail at this stage).
- manual-routing-guide.md: step-by-step KiCad GUI routing instructions
  starting with the TPS54531 buck and the AO4407A high-side switch
  per their datasheets, then digital signals, then ground stitching.

Docs updated:
- fabrication-readiness.md now lists the two routing paths and the
  validation gate.
- hardware/zero3-carrier/README.md adds the three new files to the
  file table and updates the unconnected-item count.

Auto-routers do not respect switching-supply layout rules; the buck
regulator and high-side switch sections must still be hand-routed per
TI's reference layout before exporting Gerbers.

Co-Authored-By: Claude Opus 4.7 <noreply@anthropic.com>
Routing:
- added copper zone on B.Cu, net GND
- added copper zone on F.Cu, net GND

Commit message: Route PCB end-to-end via Freerouting; export PCBWay Gerber package
PCB routing:
- route_with_freerouting.py runs end-to-end: exports Specctra DSN via
  pcbnew.ExportSpecctraDSN (KiCad 10's kicad-cli dropped that
  subcommand), invokes Freerouting v2.1.0 (pinned because v2.2.x
  requires Java 25), imports the SES via pcbnew.ImportSpecctraSES,
  refills the GND pour, and re-runs DRC.
- Freerouting pass converged in 4 passes at the 'medium' effort setting
  with zero unrouted nets.
- Final state: ERC 0, DRC 0, unconnected items 0.

Fabrication package (hardware/zero3-carrier/fabrication/):
- pcbway/zero3-water-logger-carrier-{F_Cu,B_Cu,F_Mask,B_Mask,
  F_Silkscreen,B_Silkscreen,Edge_Cuts}.* and .drl + drill map +
  drill report + .gbrjob + schematic.pdf.
- pcbway/REVIEW-BEFORE-ORDER.md: manual checklist that must clear
  before ordering, with the TPS54531 buck and AO4407A high-side
  switch routing being the most critical items (auto-routers do not
  follow switching-supply datasheet layout rules).
- zero3-water-logger-carrier-R1.zip: the entire pcbway/ folder
  packaged for upload.

.gitignore:
- DSN, SES, freerouting-run.log, freerouting.json are regenerable
  artefacts; excluded.

Docs:
- README.md and fabrication-readiness.md reflect the new
  "Gerbers exported, review-before-order" state.

Co-Authored-By: Claude Opus 4.7 <noreply@anthropic.com>
Routing:
- net OPI_5V_SW: track 0.00 -> 498.0 mm, vias 0 -> 1
- net OPI_3V3: track 0.00 -> 399.1 mm, vias 0 -> 3
- net FUSED_5V1: track 0.00 -> 303.8 mm, vias 0 -> 3
- net OPI_SCL: track 0.00 -> 237.7 mm, vias 0 -> 3
- net OPI_SDA: track 0.00 -> 224.9 mm
- net PICO_GP15: track 0.00 -> 218.6 mm, vias 0 -> 1
- net PICO_GP5: track 0.00 -> 207.1 mm, vias 0 -> 2
- net PD_FUSED: track 0.00 -> 204.5 mm, vias 0 -> 2
- net PICO_LED_GP16: track 0.00 -> 202.2 mm, vias 0 -> 2
- net OPI_1WIRE: track 0.00 -> 201.4 mm
- net PICO_GP4: track 0.00 -> 195.9 mm
- net PICO_GP14: track 0.00 -> 195.8 mm, vias 0 -> 1
- net PICO_3V3: track 0.00 -> 191.1 mm
- net PH_AIN: track 0.00 -> 178.6 mm, vias 0 -> 1
- net SPARE_AIN3: track 0.00 -> 159.9 mm, vias 0 -> 1
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