File: hardware/zero3-carrier/zero3-water-logger-carrier.kicad_sch (KiCad schematic)
At the start: 0 parts

Commit message: Add schematic synced Zero 3 carrier PCB draft
Parts:
- added C1: 470uF-1000uF 10V, Capacitor_THT:CP_Radial_D10.0mm_P5.00mm, symbol WL:C1
- added CBOOT: 100nF, Capacitor_SMD:C_0603_1608Metric, symbol WL:CBOOT
- added CCOMP1: 2200pF, Capacitor_SMD:C_0603_1608Metric, symbol WL:CCOMP1
- added CCOMP2: 22pF, Capacitor_SMD:C_0603_1608Metric, symbol WL:CCOMP2
- added CIN1: 4.7uF 50V, Capacitor_SMD:C_1206_3216Metric, symbol WL:CIN1
- added CIN2: 4.7uF 50V, Capacitor_SMD:C_1206_3216Metric, symbol WL:CIN2
- added CIN3: 10nF 50V, Capacitor_SMD:C_0603_1608Metric, symbol WL:CIN3
- added COUT1: 47uF 10V, Capacitor_SMD:C_1210_3225Metric, symbol WL:COUT1
- added COUT2: 47uF 10V, Capacitor_SMD:C_1210_3225Metric, symbol WL:COUT2
- added CSS: 10nF, Capacitor_SMD:C_0603_1608Metric, symbol WL:CSS
- added D1: VBUS TVS, Diode_SMD:D_SMA, symbol WL:D1
- added D2: 5A 40V Schottky, Diode_SMD:D_SMA, symbol WL:D2
- added F1: 3A-5A polyfuse, Fuse:Fuse_1206_3216Metric, symbol WL:F1
- added J1: Orange Pi Zero 3 26-pin, Connector_PinHeader_2.54mm:PinHeader_2x13_P2.54mm_Vertical, symbol WL:J1
- added J10: Turbidity sensor, TerminalBlock_Phoenix:TerminalBlock_Phoenix_MKDS-1,5-3-5.08_1x03_P5.08mm_Horizontal, symbol WL:J10
- added J11: ORP sensor, TerminalBlock_Phoenix:TerminalBlock_Phoenix_MKDS-1,5-3-5.08_1x03_P5.08mm_Horizontal, symbol WL:J11
- added J12: Dissolved oxygen, TerminalBlock_Phoenix:TerminalBlock_Phoenix_MKDS-1,5-3-5.08_1x03_P5.08mm_Horizontal, symbol WL:J12
- added J13: NH4 ISE amp, TerminalBlock_Phoenix:TerminalBlock_Phoenix_MKDS-1,5-3-5.08_1x03_P5.08mm_Horizontal, symbol WL:J13
- added J14: USB-C PD input, Connector_USB:USB_C_Receptacle_HRO_TYPE-C-31-M-12, symbol WL:J14
- added J15: Download button, Connector_PinHeader_2.54mm:PinHeader_1x04_P2.54mm_Vertical, symbol WL:J15
- added J16: Spare analog header, Connector_PinHeader_2.54mm:PinHeader_1x04_P2.54mm_Vertical, symbol WL:J16
- added J2: Raspberry Pi Pico socket, Module:RaspberryPi_Pico_Common_THT, symbol WL:J2
- added J3: ADS1115 #1 0x48, Connector_PinHeader_2.54mm:PinHeader_1x09_P2.54mm_Vertical, symbol WL:J3
- added J4: ADS1115 #2 0x49, Connector_PinHeader_2.54mm:PinHeader_1x09_P2.54mm_Vertical, symbol WL:J4
- added J5: DS18B20 water temp, Connector_PinHeader_2.54mm:PinHeader_1x03_P2.54mm_Vertical, symbol WL:J5
- added J6: BME280 air sensor, Connector_PinHeader_2.54mm:PinHeader_1x04_P2.54mm_Vertical, symbol WL:J6
- added J7: DS3231 RTC, Connector_PinHeader_2.54mm:PinHeader_1x04_P2.54mm_Vertical, symbol WL:J7
- added J8: pH sensor, TerminalBlock_Phoenix:TerminalBlock_Phoenix_MKDS-1,5-3-5.08_1x03_P5.08mm_Horizontal, symbol WL:J8
- added J9: TDS sensor, TerminalBlock_Phoenix:TerminalBlock_Phoenix_MKDS-1,5-3-5.08_1x03_P5.08mm_Horizontal, symbol WL:J9
- added L1: 4.7uH >=6A, Inductor_SMD:L_10.4x10.4_H4.8, symbol WL:L1
- added Q1: AO4407A P-MOS high-side, Package_SO:SOIC-8_3.9x4.9mm_P1.27mm, symbol WL:Q1
- added Q2: 2N7002, Package_TO_SOT_SMD:SOT-23, symbol WL:Q2
- added R1: 4.7k, Resistor_THT:R_Axial_DIN0207_L6.3mm_D2.5mm_P7.62mm_Horizontal, symbol WL:R1
- added R2: 100k, Resistor_SMD:R_0603_1608Metric, symbol WL:R2
- added R3: 1k, Resistor_SMD:R_0603_1608Metric, symbol WL:R3
- added R4: 100k, Resistor_SMD:R_0603_1608Metric, symbol WL:R4
- added R5: 330R if 3.3V LED, Resistor_SMD:R_0603_1608Metric, symbol WL:R5
- added RCOMP1: 37.4k, Resistor_SMD:R_0603_1608Metric, symbol WL:RCOMP1
- added REN1: 665k, Resistor_SMD:R_0603_1608Metric, symbol WL:REN1
- added REN2: 130k, Resistor_SMD:R_0603_1608Metric, symbol WL:REN2
- added RFB1: 10.2k 1%, Resistor_SMD:R_0603_1608Metric, symbol WL:RFB1
- added RFB2: 1.96k 1%, Resistor_SMD:R_0603_1608Metric, symbol WL:RFB2
- added U1: CH224K PD sink 9V, Package_SO:SSOP-10_3.9x4.9mm_P1.00mm, symbol WL:U1
- added U2: TPS54531DDA 5A buck, Package_SO:TI_SO-PowerPAD-8, symbol WL:U2
Connections:
- new net BUCK_BOOT: CBOOT.1 (BOOT), U2.BOOT
- new net BUCK_COMP: CCOMP2.1 (COMP), RCOMP1.1 (COMP), U2.COMP
- new net BUCK_COMP_RC: CCOMP1.1 (NODE), RCOMP1.2 (NODE)
- new net BUCK_EN: REN1.2 (EN), REN2.1 (EN), U2.EN
- new net BUCK_FB: RFB1.2 (FB), RFB2.1 (FB), U2.VSENSE (FB)
- new net BUCK_SS: CSS.1 (SS), U2.SS
- new net BUCK_SW: CBOOT.2 (SW), D2.K, L1.1 (SW), U2.PH (PH/SW)
- new net BUTTON_LED_A: J15.3 (LED+), R5.2 (LED+)
- new net DO_AIN: J12.3 (AO), J4.6 (A0)
- new net FUSED_5V1: COUT1.1 (+), COUT2.1 (+), J2.39 (VSYS), L1.2 (OUT), Q1.S (SOURCE), R2.1 (5V1), RFB1.1 (TOP)
- new net GND: C1.2 (-), CCOMP1.2 (GND), CCOMP2.2 (GND), CIN1.2 (-), CIN2.2 (-), CIN3.2 (-), COUT1.2 (-), COUT2.2 (-), CSS.2 (GND), D1.2 (A), D2.A, J1.14 (GND), J1.20 (GND), J1.25 (GND), J1.6 (GND), J1.9 (GND), J10.2 (GND), J11.2 (GND), J12.2 (GND), J13.2 (GND), J14.A1/B1/A12/B12 (GND), J14.SH (SHIELD), J15.2 (C), J15.4 (LED-), J16.2 (GND), J2.13 (GND), J2.18 (GND), J2.23 (GND), J2.28 (GND), J2.3 (GND), J2.33 (GND), J2.38 (GND), J2.8 (GND), J3.2 (GND), J3.5 (ADDR), J4.2 (GND), J5.3 (GND), J6.2 (GND), J7.2 (GND), J8.2 (GND), J9.2 (GND), Q2.S (SOURCE), R4.2 (GND), REN2.2 (GND), RFB2.2 (GND), U1.GND, U2.GND, U2.PAD (EP)
- new net NH4_AIN: J13.3 (AO), J4.7 (A1)
- new net OPI_1WIRE: J1.7 (1WIRE), J5.2 (DATA), R1.2 (DATA)
- new net OPI_3V3: J1.1 (3V3), J1.17 (3V3), J16.1 (3V3), J3.1 (VDD), J4.1 (VDD), J4.5 (ADDR), J5.1 (VCC), J6.1 (VCC), R1.1 (3V3)
- new net OPI_5V_SW: C1.1 (+), J1.2 (5V), J1.4 (5V), J10.1 (5V), J11.1 (5V), J12.1 (5V), J13.1 (5V), J8.1 (5V), J9.1 (5V), Q1.D (DRAIN)
- new net OPI_READY: J1.11 (READY), J2.17 (GP13)
- new net OPI_SCL: J1.5 (SCL), J3.4 (SCL), J4.4 (SCL), J6.4 (SCL)
- new net OPI_SDA: J1.3 (SDA), J3.3 (SDA), J4.3 (SDA), J6.3 (SDA)
- new net ORP_AIN: J11.3 (AO), J3.9 (A3)
- new net PD_CFG: U1.CFG1, U1.CFG2, U1.CFG3
- new net PD_FUSED: CIN1.1 (+), CIN2.1 (+), CIN3.1 (+), F1.2 (OUT), REN1.1 (VIN), U2.VIN
- new net PD_NEGOTIATED_VBUS: F1.1 (IN), U1.VOUT
- new net PH_AIN: J3.6 (A0), J8.3 (AO)
- new net PICO_3V3: J2.36 (3V3), J7.1 (VCC)
- new net PICO_GP14: J15.1 (NO), J2.19 (GP14)
- new net PICO_GP15: J2.20 (GP15), R3.1 (PICO)
- new net PICO_GP4: J2.6 (GP4), J7.3 (SDA)
- new net PICO_GP5: J2.7 (GP5), J7.4 (SCL)
- new net PICO_LED_GP16: J2.21 (GP16/LED), R5.1 (PICO)
- new net PWR_GATE: Q1.G (GATE), Q2.D (DRAIN), R2.2 (GATE)
- new net Q2_GATE: Q2.G (GATE), R3.2 (Q2G), R4.1 (Q2G)
- new net SPARE_AIN2: J16.3 (AIN2), J4.8 (A2)
- new net SPARE_AIN3: J16.4 (AIN3), J4.9 (A3)
- new net TDS_AIN: J3.7 (A1), J9.3 (AO)
- new net TURB_AIN: J10.3 (AO), J3.8 (A2)
- new net UART_OPI_TX_PICO_RX: J1.8 (TX), J2.2 (GP1/RX)
- new net UART_PICO_TX_OPI_RX: J1.10 (RX), J2.1 (GP0/TX)
- new net USB_CC1: J14.A5 (CC1), U1.CC1
- new net USB_CC2: J14.B5 (CC2), U1.CC2
- new net USB_VBUS: D1.1 (K), J14.A4/B4/A9/B9 (VBUS), U1.VBUS
Other:
- note added: "Buck regulator PCB layout must follow TPS54531 datasheet: short SW loop, thermal copper, tight input caps."
- note added: "Pico is always-on from FUSED_5V1. Orange Pi and wet-side sensor 5V are switched by Q1."
- note added: "USB-C PD front end: CH224K requests 9V, TPS54531 generates protected 5.1V."
- note added: "Verify CH224K strap pins and all package pinouts against supplier datasheets before PCB order."
- note removed: "R0 KiCad project scaffold. Build the final schematic from zero3-water-logger-carrier-pinout.csv before ordering."
